Commit message: Update Capsule_robot.urdf

File: Capsule_robot_description/urdf/Capsule_robot.urdf (robot description, URDF)
Before this commit: robot Capsule_robot, 10 links, 9 joints
Links:
- link Capsule10_1: geometry collision mesh filename=../meshes/Capsule10_1.stl scale=0.001 0.001 0.001; visual mesh filename=../meshes/Capsule10_1.stl scale=0.001 0.001 0.001
- link Capsule2_1: geometry collision mesh filename=../meshes/Capsule2_1.stl scale=0.001 0.001 0.001; visual mesh filename=../meshes/Capsule2_1.stl scale=0.001 0.001 0.001
- link Capsule3_1: geometry collision mesh filename=../meshes/Capsule3_1.stl scale=0.001 0.001 0.001; visual mesh filename=../meshes/Capsule3_1.stl scale=0.001 0.001 0.001
- link Capsule4_1: geometry collision mesh filename=../meshes/Capsule4_1.stl scale=0.001 0.001 0.001; visual mesh filename=../meshes/Capsule4_1.stl scale=0.001 0.001 0.001
- link Capsule5_1: geometry collision mesh filename=../meshes/Capsule5_1.stl scale=0.001 0.001 0.001; visual mesh filename=../meshes/Capsule5_1.stl scale=0.001 0.001 0.001
- link Capsule6_1: geometry collision mesh filename=../meshes/Capsule6_1.stl scale=0.001 0.001 0.001; visual mesh filename=../meshes/Capsule6_1.stl scale=0.001 0.001 0.001
- link Capsule7_1: geometry collision mesh filename=../meshes/Capsule7_1.stl scale=0.001 0.001 0.001; visual mesh filename=../meshes/Capsule7_1.stl scale=0.001 0.001 0.001
- link Capsule8_1: geometry collision mesh filename=../meshes/Capsule8_1.stl scale=0.001 0.001 0.001; visual mesh filename=../meshes/Capsule8_1.stl scale=0.001 0.001 0.001
- link Capsule9_1: geometry collision mesh filename=../meshes/Capsule9_1.stl scale=0.001 0.001 0.001; visual mesh filename=../meshes/Capsule9_1.stl scale=0.001 0.001 0.001
- link base_link: geometry collision mesh filename=../meshes/base_link.stl scale=0.001 0.001 0.001; visual mesh filename=../meshes/base_link.stl scale=0.001 0.001 0.001
